File: zx81-external-16k.kicad_pcb (KiCad board)
At the start: 2 copper layers, 59.8 x 42.7 mm, 14 parts, among them J1 Connector ZX81, U1 CY62256-70PC, U2 74LS00, U3 74LS32

Commit message: KiCad update
Parts:
- added D4: 1N4148, Diode_THT:D_DO-35_SOD27_P7.62mm_Horizontal, F.Cu at (129.4, 112.1)
- moved D2 2.31 mm to (117.9, 112.2)
- moved D3 1.36 mm to (106.9, 112.2)
Connections:
- J1 pad A25: Net-(J1-~{ROMCS}) -> Net-(D4-K)
- U2 pad 4: Net-(J1-~{ROMCS}) -> Net-(D4-A)
- U3 pad 3: Net-(J1-~{ROMCS}) -> Net-(D4-A)
Routing:
- net Net-(J1-~{ROMCS}): track 39.4 -> 0.00 mm
- net Net-(D4-K): track 0.00 -> 37.7 mm, vias 0 -> 1
- net Net-(D4-A): track 0.00 -> 24.9 mm
- net +5V: track 127.0 -> 104.6 mm, vias 0 -> 1
- net A7: track 78.9 -> 61.3 mm, vias 1 -> 3
- net Net-(D2-K): track 68.8 -> 54.1 mm, vias 2 -> 0
- net D5: track 40.7 -> 54.4 mm, vias 2 -> 3
- net A10: track 40.2 -> 53.6 mm, vias 0 -> 2
- net A3: track 33.1 -> 21.6 mm
- net A13: track 44.8 -> 56.2 mm, vias 1 -> 2
- net D4: track 44.4 -> 34.7 mm, vias 1 -> 3
- net A11: track 40.1 -> 48.9 mm, vias 0 -> 2
- net A0: track 20.9 -> 29.4 mm, vias 1 -> 0
- net Net-(J1-~{WR}): track 65.1 -> 73.3 mm, vias 1 -> 4
- net A15: track 43.3 -> 50.2 mm
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Other:
- board text added: "ZX81 16/32K RAM v1.2 - by ZXINFO"
- board text removed: "ZX81 16/32K RAM v1.1 - by ZXINFO"
