File: zx81-external-16k.kicad_sch (KiCad schematic)
At the start: 14 parts, among them J1 Connector ZX81, U1 CY62256-70PC, U2 74LS00, U3 74LS32

Commit message: KiCad update
Parts:
- added D4: 1N4148, Diode_THT:D_DO-35_SOD27_P7.62mm_Horizontal, symbol Diode:1N4148
Connections:
- net at U2.4, U3.3: now also D4.2 (A); no longer J1.A25 (~{ROMCS})
- new net: D4.1 (K), J1.A25 (~{ROMCS})
Other:
- title: ZX81 external 16Kb RAM - Simple -> ZX81 external 32Kb RAM
Changed lines of the file:
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@@
 (kicad_sch
-	(version 20231120)
+	(version 20250114)
 	(generator "eeschema")
-	(generator_version "8.0")
+	(generator_version "9.0")
 	(paper "A4")
 	(title_block
-		(title "ZX81 external 16Kb RAM - Simple")
+		(title "ZX81 external 32Kb RAM")
 		(date "2024-04-23")
-		(rev "v1")
+		(rev "v1.2")
 		(company "ZXInfo")
 	)
+	(text_box "ZX81 external 16Kb RAM in a very simple version.\n\nv1.1\n- R footprint a little bigger\n- M1not logic to control extra 16K RAM from 32K to 48K\n- Jumper to enable 32K - 32K to 48K\n- ROM disabled when accessing RAM 16-48K\n- Address logic for MREQ + (A14 or A15) -> CS\n- Added capacitor between PIN 20 and GND for WRX\n\nv1.0\n- Internal RAM always disabled by RAMCS high\n- WR -> WE (write enable)\n- RD -> OE(out enable)\n- MREQ + A14 -> CS\n"
+		(exclude_from_sim no)
+		(at 190.5 15.24 0)
+		(size 90.17 52.07)
+		(margins 1.35 1.35 1.35 1.35)
+		(stroke
+			(width 0)
+			(type dash)
+		)
+		(fill
+			(type none)
+		)
+		(effects
+			(font
+				(size 1.8 1.8)
+			)
+			(justify left top)
+		)
+	)
 	(junction
 		(at 228.6 102.87)
@@
 	(wire
 		(pts
-			(xy 191.77 97.79) (xy 191.77 102.87)
+			(xy 97.79 93.98) (xy 105.41 93.98)
 		)
 		(stroke
@@
 	(wire
 		(pts
-			(xy 191.77 102.87) (xy 191.77 114.3)
+			(xy 191.77 97.79) (xy 191.77 102.87)
 		)
 		(stroke
@@
 	(wire
 		(pts
-			(xy 81.28 38.1) (xy 82.55 38.1)
+			(xy 191.77 102.87) (xy 191.77 114.3)
 		)
 		(stroke
@@
 	(wire
 		(pts
-			(xy 44.45 158.75) (xy 68.58 158.75)
+			(xy 81.28 38.1) (xy 82.55 38.1)
 		)
 		(stroke
@@
 	(wire
 		(pts
-			(xy 86.36 124.46) (xy 90.17 124.46)
+			(xy 44.45 158.75) (xy 68.58 158.75)
 		)
 		(stroke
@@
 	(wire
 		(pts
-			(xy 91.44 31.75) (xy 100.33 31.75)
+			(xy 86.36 124.46) (xy 90.17 124.46)
 		)
 		(stroke
@@
 	(wire
 		(pts
-			(xy 153.67 74.93) (xy 153.67 165.1)
+			(xy 91.44 31.75) (xy 100.33 31.75)
 		)
 		(stroke
@@
 	(wire
 		(pts
-			(xy 81.28 93.98) (xy 105.41 93.98)
+			(xy 153.67 74.93) (xy 153.67 165.1)
 		)
 		(stroke
@@
 	(wire
 		(pts
+			(xy 81.28 93.98) (xy 90.17 93.98)
+		)
+		(stroke
+			(width 0)
+			(type default)
+		)
+	)
+	(wire
+		(pts
 			(xy 228.6 114.3) (xy 255.27 114.3)
 		)
@@
 		)
 	)
-	(text_box "ZX81 external 16Kb RAM in a very simple version.\n\nv1.1\n- R footprint a little bigger\n- M1not logic to control extra 16K RAM from 32K to 48K\n- Jumper to enable 32K - 32K to 48K\n- ROM disabled when accessing RAM 16-48K\n- Address logic for MREQ + (A14 or A15) -> CS\n- Added capacitor between PIN 20 and GND for WRX\n\nv1.0\n- Internal RAM always disabled by RAMCS high\n- WR -> WE (write enable)\n- RD -> OE(out enable)\n- MREQ + A14 -> CS\n"
-		(exclude_from_sim no)
-		(at 190.5 15.24 0)
-		(size 90.17 52.07)
-		(stroke
-			(width 0)
-			(type dash)
-		)
-		(fill
-			(type none)
-		)
-		(effects
-			(font
-				(size 1.8 1.8)
-			)
-			(justify left top)
-		)
-	)
 	(global_label "D4"
 		(shape input)
@@
 	)
 	(symbol
+		(lib_id "Diode:1N4148")
+		(at 93.98 93.98 0)
+		(unit 1)
+		(exclude_from_sim no)
+		(in_bom yes)
+		(on_board yes)
+		(dnp no)
+		(fields_autoplaced yes)
+		(property "Reference" "D4"
+			(at 93.98 87.63 0)
+			(effects
+				(font
+					(size 1.27 1.27)
+				)
+			)
+		)
+		(property "Value" "1N4148"
+			(at 93.98 90.17 0)
+			(effects
+				(font
+					(size 1.27 1.27)
+				)
+			)
+		)
+		(property "Footprint" "Diode_THT:D_DO-35_SOD27_P7.62mm_Horizontal"
+			(at 93.98 93.98 0)
+			(effects
+				(font
+					(size 1.27 1.27)
+				)
+				(hide yes)
+			)
+		)
+		(property "Datasheet" "https://assets.nexperia.com/documents/data-sheet/1N4148_1N4448.pdf"
+			(at 93.98 93.98 0)
+			(effects
+				(font
+					(size 1.27 1.27)
+				)
+				(hide yes)
+			)
+		)
+		(property "Description" "100V 0.15A standard switching diode, DO-35"
+			(at 93.98 93.98 0)
+			(effects
+				(font
+					(size 1.27 1.27)
+				)
+				(hide yes)
+			)
+		)
+		(property "Sim.Device" "D"
+			(at 93.98 93.98 0)
+			(effects
+				(font
+					(size 1.27 1.27)
+				)
+				(hide yes)
+			)
+		)
+		(property "Sim.Pins" "1=K 2=A"
+			(at 93.98 93.98 0)
+			(effects
+				(font
+					(size 1.27 1.27)
+				)
+				(hide yes)
+			)
+		)
+		(pin "1"
+		)
+		(pin "2"
+		)
+		(instances
+			(project ""
+				(path "/51054ebb-4879-470e-b753-9ec62a0d0736"
+					(reference "D4")
+					(unit 1)
+				)
+			)
+		)
+	)
+	(symbol
 		(lib_id "Device:R")
 		(at 78.74 172.72 180)
@@
 		)
 	)
+	(embedded_fonts no)
 )
